Commit message: Phase 5: Implement FPV Cockpit - Camera driver, Dashboard feed, and Auto-Launch service

File: rover1_description/urdf/rover.urdf.xacro (robot description, xacro)
@@ -79,7 +79,20 @@
     </joint>
   </xacro:macro>
-  <xacro:wheel prefix="front_left" x="0.1" y="0.12"/>
-  <xacro:wheel prefix="front_right" x="0.1" y="-0.12"/>
-  <xacro:wheel prefix="rear_left" x="-0.1" y="0.12"/>
   <xacro:wheel prefix="rear_right" x="-0.1" y="-0.12"/>
+  <!-- Camera Link (Nuwa-HP60C) -->
+  <link name="camera_link">
+    <visual>
+      <geometry>
+        <box size="0.05 0.05 0.05"/>
+      </geometry>
+      <material name="black"/>
+    </visual>
+  </link>
+  <joint name="camera_joint" type="fixed">
+    <parent link="base_link"/>
+    <child link="camera_link"/>
+    <!-- Position: Near front (0.12m), Height: 33cm from ground (24cm from center) -->
+    <!-- Orientation: 7 degrees downward pitch (0.122 radians) -->
+    <origin xyz="0.12 0 0.24" rpy="0 0.122 0"/>
+  </joint>
 </robot>

Commit message: Fix: Optimize dashboard event loop, fix camera config paths, and add optical frame

File: rover1_description/urdf/rover.urdf.xacro (robot description, xacro)
@@ -96,3 +96,10 @@
     <origin xyz="0.12 0 0.24" rpy="0 0.122 0"/>
   </joint>
+  <!-- Optical frame for standard vision processing (Z forward, X right, Y down) -->
+  <link name="camera_optical_frame"/>
+  <joint name="camera_optical_joint" type="fixed">
+    <parent link="camera_link"/>
+    <child link="camera_optical_frame"/>
+    <origin xyz="0 0 0" rpy="-${pi/2} 0 -${pi/2}"/>
+  </joint>
 </robot>
